File: PCB/HUB75_Driver.sch (KiCad schematic (older format))
At the start: 15 parts, among them U1 ESP32_DevKit_V1_DOIT

Commit message: add reset capacitor
Parts:
- added C_PROG_1: 10uF, Capacitor_SMD:C_0603_1608Metric, symbol Device:C
Connections:
- net GND: now also C_PROG_1.2
- net at U1.1 (EN): now also C_PROG_1.1
- no-connect marks 2 -> 8
Other:
- moved on the sheet: F1
Changed lines of the file:
@@
 U 1 1 61B3A49D
 P 1700 1250
-F 0 "J_IN_1" H 1618 1467 50  0000 C CNN
-F 1 "Screw_Terminal_01x02" H 1618 1376 50  0000 C CNN
+F 0 "J_IN_1" H 1800 1450 50  0000 C CNN
+F 1 "Screw_Terminal_01x02" H 1800 1350 50  0000 C CNN
 F 2 "TerminalBlock:TerminalBlock_bornier-2_P5.08mm" H 1700 1250 50  0001 C CNN
 F 3 "~" H 1700 1250 50  0001 C CNN
@@
 L Device:Polyfuse F1
 U 1 1 61B3DBC0
-P 2250 1250
-F 0 "F1" V 2475 1250 50  0000 C CNN
-F 1 "5A" V 2384 1250 50  0000 C CNN
-F 2 "Fuse:Fuse_0805_2012Metric_Pad1.15x1.40mm_HandSolder" H 2300 1050 50  0001 L CNN
-F 3 "~" H 2250 1250 50  0001 C CNN
-	1    2250 1250
+P 2150 1250
+F 0 "F1" V 2375 1250 50  0000 C CNN
+F 1 "5A" V 2284 1250 50  0000 C CNN
+F 2 "Fuse:Fuse_0805_2012Metric_Pad1.15x1.40mm_HandSolder" H 2200 1050 50  0001 L CNN
+F 3 "~" H 2150 1250 50  0001 C CNN
+	1    2150 1250
 	0    -1   -1   0
 $EndComp
@@
 L power:PWR_FLAG #FLG0101
 U 1 1 61B3FB22
-P 2000 1250
-F 0 "#FLG0101" H 2000 1325 50  0001 C CNN
-F 1 "PWR_FLAG" H 2000 1423 50  0001 C CNN
-F 2 "" H 2000 1250 50  0001 C CNN
-F 3 "~" H 2000 1250 50  0001 C CNN
-	1    2000 1250
+P 2450 1250
+F 0 "#FLG0101" H 2450 1325 50  0001 C CNN
+F 1 "PWR_FLAG" H 2450 1423 50  0001 C CNN
+F 2 "" H 2450 1250 50  0001 C CNN
+F 3 "~" H 2450 1250 50  0001 C CNN
+	1    2450 1250
 	1    0    0    -1
 $EndComp
@@
 L power:PWR_FLAG #FLG0102
 U 1 1 61B401F6
-P 2000 1350
-F 0 "#FLG0102" H 2000 1425 50  0001 C CNN
-F 1 "PWR_FLAG" H 2000 1523 50  0001 C CNN
-F 2 "" H 2000 1350 50  0001 C CNN
-F 3 "~" H 2000 1350 50  0001 C CNN
-	1    2000 1350
+P 2450 1350
+F 0 "#FLG0102" H 2450 1425 50  0001 C CNN
+F 1 "PWR_FLAG" H 2450 1523 50  0001 C CNN
+F 2 "" H 2450 1350 50  0001 C CNN
+F 3 "~" H 2450 1350 50  0001 C CNN
+	1    2450 1350
 	-1   0    0    1
 $EndComp
 Wire Wire Line
 	1900 1250 2000 1250
-Connection ~ 2000 1250
-Wire Wire Line
-	2000 1250 2100 1250
-Wire Wire Line
-	1900 1350 2000 1350
-Connection ~ 2000 1350
-Wire Wire Line
-	2400 1250 2550 1250
+Wire Wire Line
+	2300 1250 2450 1250
 Connection ~ 2550 1250
 Wire Wire Line
@@
 Connection ~ 2550 1350
 Wire Wire Line
-	2000 1350 2550 1350
+	1900 1350 2450 1350
 $Comp
 L power:+5V #PWR0103
@@
 Connector_IDC:IDC-Header_2x08_P2.54mm_Vertical
 Wire Wire Line
-	2250 3300 2250 3000
+	2250 3300 2250 3250
 $Comp
 L Graphic:Logo_Open_Hardware_Small LOGO1
@@
 	1    0    0    -1
 $EndComp
+NoConn ~ 2850 3600
+NoConn ~ 2850 3800
+NoConn ~ 2850 5700
+NoConn ~ 2850 5800
+NoConn ~ 2850 4600
+NoConn ~ 2850 4500
+$Comp
+L Device:C C_PROG_1
+U 1 1 61B8E21E
+P 1150 3650
+F 0 "C_PROG_1" H 1265 3696 50  0000 L CNN
+F 1 "10uF" H 1265 3605 50  0000 L CNN
+F 2 "Capacitor_SMD:C_0603_1608Metric" H 1188 3500 50  0001 C CNN
+F 3 "~" H 1150 3650 50  0001 C CNN
+	1    1150 3650
+	1    0    0    -1
+$EndComp
+Wire Wire Line
+	1650 3500 1150 3500
+$Comp
+L power:GND #PWR0109
+U 1 1 61B8ECFD
+P 1150 3800
+F 0 "#PWR0109" H 1150 3550 50  0001 C CNN
+F 1 "GND" H 1155 3627 50  0000 C CNN
+F 2 "" H 1150 3800 50  0001 C CNN
+F 3 "" H 1150 3800 50  0001 C CNN
+	1    1150 3800
+	1    0    0    -1
+$EndComp
+Connection ~ 2450 1250
+Wire Wire Line
+	2450 1250 2550 1250
+Connection ~ 2450 1350
+Wire Wire Line
+	2450 1350 2550 1350
+$Comp
+L power:PWR_FLAG #FLG0103
+U 1 1 61B91850
+P 2250 3250
+F 0 "#FLG0103" H 2250 3325 50  0001 C CNN
+F 1 "PWR_FLAG" H 2250 3423 50  0001 C CNN
+F 2 "" H 2250 3250 50  0001 C CNN
+F 3 "~" H 2250 3250 50  0001 C CNN
+	1    2250 3250
+	0    1    1    0
+$EndComp
+Connection ~ 2250 3250
+Wire Wire Line
+	2250 3250 2250 3000
+$Comp
+L power:PWR_FLAG #FLG0104
+U 1 1 61B91E58
+P 2150 2600
+F 0 "#FLG0104" H 2150 2675 50  0001 C CNN
+F 1 "PWR_FLAG" H 2150 2773 50  0001 C CNN
+F 2 "" H 2150 2600 50  0001 C CNN
+F 3 "~" H 2150 2600 50  0001 C CNN
+	1    2150 2600
+	0    1    1    0
+$EndComp
+Connection ~ 2150 2600
 $EndSCHEMATC
